File: kicad_docs/CV_path.sch (KiCad schematic (older format))
At the start: 21 parts, among them U4 TL072

Commit message: first rev pcb layout
Other:
- note added: "approximately\n+2 volts to 0 volts"
- note added: "approximately\n0 volts to +1 volts"
- note removed: "+2 volts to 0 volts"
- note removed: "0 volts to +1 volts"
Changed lines of the file:
@@
 	0    1    1    0
 $EndComp
-Text Notes 9800 3800 0    50   ~ 0
-0 volts to +1 volts
-Text Notes 4200 4900 0    50   ~ 0
-+2 volts to 0 volts
+Text Notes 9800 3850 0    50   ~ 0
+approximately\n0 volts to +1 volts
+Text Notes 4150 4950 0    50   ~ 0
+approximately\n+2 volts to 0 volts
 $EndSCHEMATC
