File: kicad_docs/2164SVF.kicad_pcb (KiCad board)
At the start: 2 copper layers, 0 parts

Commit message: first rev pcb layout
Parts:
- added C1: 47pF, Capacitor_SMD:C_0805_2012Metric_Pad1.15x1.40mm_HandSolder, B.Cu at (126.5, 70.9)
- added C10: 100nF, Capacitor_SMD:C_0805_2012Metric_Pad1.15x1.40mm_HandSolder, B.Cu at (115.3, 63.5)
- added C11: 100pF, Capacitor_SMD:C_0805_2012Metric_Pad1.15x1.40mm_HandSolder, B.Cu at (133.6, 124.7)
- added C12: 100nF, Capacitor_SMD:C_0805_2012Metric_Pad1.15x1.40mm_HandSolder, B.Cu at (148.8, 63.2)
- added C13: 100pF, Capacitor_SMD:C_0805_2012Metric_Pad1.15x1.40mm_HandSolder, B.Cu at (147.8, 121.7)
- added C14: 10uF, Capacitor_SMD:CP_Elec_6.3x5.4_Nichicon, B.Cu at (120.8, 52.8)
- added C15: 10uF, Capacitor_SMD:CP_Elec_6.3x5.4_Nichicon, B.Cu at (144.7, 52.8)
- added C16: 100nF, Capacitor_SMD:C_0805_2012Metric_Pad1.15x1.40mm_HandSolder, B.Cu at (152.1, 69.3)
- added C17: 100nF, Capacitor_SMD:C_0805_2012Metric_Pad1.15x1.40mm_HandSolder, B.Cu at (128.5, 80.3)
- added C18: 100nF, Capacitor_SMD:C_0805_2012Metric_Pad1.15x1.40mm_HandSolder, B.Cu at (128.5, 76.2)
- added C19: 100nF, Capacitor_SMD:C_0805_2012Metric_Pad1.15x1.40mm_HandSolder, B.Cu at (116.8, 80.3)
- added C2: 100pF, Capacitor_SMD:C_0805_2012Metric_Pad1.15x1.40mm_HandSolder, B.Cu at (109.2, 70.9)
- added C20: 100nF, Capacitor_SMD:C_0805_2012Metric_Pad1.15x1.40mm_HandSolder, B.Cu at (116.8, 76.2)
- added C21: 100nF, Capacitor_SMD:C_0805_2012Metric_Pad1.15x1.40mm_HandSolder, B.Cu at (106.4, 80.3)
- added C22: 100nF, Capacitor_SMD:C_0805_2012Metric_Pad1.15x1.40mm_HandSolder, B.Cu at (106.4, 76.2)
- added C23: 100nF, Capacitor_SMD:C_0805_2012Metric_Pad1.15x1.40mm_HandSolder, B.Cu at (152.1, 74.2)
- added C24: 100nF, Capacitor_SMD:C_0805_2012Metric_Pad1.15x1.40mm_HandSolder, B.Cu at (142.7, 114.6)
- added C25: 100nF, Capacitor_SMD:C_0805_2012Metric_Pad1.15x1.40mm_HandSolder, B.Cu at (138.7, 114.6)
- added C3: 560pF, Capacitor_SMD:C_0805_2012Metric_Pad1.15x1.40mm_HandSolder, B.Cu at (132.1, 70.9)
- added C4: 560pF, Capacitor_SMD:C_0805_2012Metric_Pad1.15x1.40mm_HandSolder, B.Cu at (135.9, 85.4)
- added C5: 22nF, svf_footprints:timing_cap_dual_fp, B.Cu at (121.3, 96.5)
- added C6: 220pF, svf_footprints:timing_cap_dual_fp, B.Cu at (120.0, 86.0)
- added C7: 560pF, Capacitor_SMD:C_0805_2012Metric_Pad1.15x1.40mm_HandSolder, B.Cu at (146.1, 70.9)
- added C8: 22nF, svf_footprints:timing_cap_dual_fp, B.Cu at (107.3, 96.5)
- added C9: 220pF, svf_footprints:timing_cap_dual_fp, B.Cu at (110.1, 86.0)
- added D1: 6z2, Diode_SMD:D_SOD-123, B.Cu at (124.0, 100.6)
- added D2: 6z2, Diode_SMD:D_SOD-123, B.Cu at (121.4, 100.6)
- added D3: 1N4148W, Diode_SMD:D_SOD-123, B.Cu at (133.1, 118.1)
- added D4: 1N4148W, Diode_SMD:D_SOD-123, B.Cu at (133.1, 121.7)
- added D5: BAT48, Diode_SMD:D_SOD-123, B.Cu at (148.3, 124.7)
- added D6: BAT48, Diode_SMD:D_SOD-123, B.Cu at (152.1, 51.2)
- added H1: MountingHole_Pad, MountingHole:MountingHole_3.2mm_M3_Pad_Via, F.Cu at (108.0, 52.1)
- added H2: MountingHole_Pad, MountingHole:MountingHole_3.2mm_M3_Pad_Via, F.Cu at (108.0, 141.0)
- added J1: PJ301M-12, svf_footprints:PJ301M-12, F.Cu at (111.1, 127.0)
- added J2: PJ301M-12, svf_footprints:PJ301M-12, F.Cu at (125.1, 127.0)
- added J3: PJ301M-12, svf_footprints:PJ301M-12, F.Cu at (139.1, 127.0)
- added J4: power_in, Connector_PinHeader_2.54mm:PinHeader_2x05_P2.54mm_Vertical, B.Cu at (133.3, 54.6)
- added J5: PJ301M-12, svf_footprints:PJ301M-12, F.Cu at (153.0, 127.0)
- added J6: PJ301M-12, svf_footprints:PJ301M-12, F.Cu at (153.0, 141.0)
- added J7: PJ301M-12, svf_footprints:PJ301M-12, F.Cu at (139.1, 141.0)
- added J8: PJ301M-12, svf_footprints:PJ301M-12, F.Cu at (125.1, 141.0)
- added R1: 1k, Resistor_SMD:R_0805_2012Metric_Pad1.15x1.40mm_HandSolder, B.Cu at (148.1, 137.4)
- added R10: 30k, Resistor_SMD:R_0805_2012Metric_Pad1.15x1.40mm_HandSolder, B.Cu at (137.7, 70.9)
- added R11: 510, Resistor_SMD:R_0805_2012Metric_Pad1.15x1.40mm_HandSolder, B.Cu at (134.9, 70.9)
- added R12: 510, Resistor_SMD:R_0805_2012Metric_Pad1.15x1.40mm_HandSolder, B.Cu at (133.1, 85.3)
- added R13: 30k, Resistor_SMD:R_0805_2012Metric_Pad1.15x1.40mm_HandSolder, B.Cu at (130.3, 85.4)
- added R14: 30k, Resistor_SMD:R_0805_2012Metric_Pad1.15x1.40mm_HandSolder, B.Cu at (140.5, 70.9)
- added R15: 510, Resistor_SMD:R_0805_2012Metric_Pad1.15x1.40mm_HandSolder, B.Cu at (143.3, 70.9)
- added R16: 100k, Resistor_SMD:R_0805_2012Metric_Pad1.15x1.40mm_HandSolder, B.Cu at (133.6, 106.4)
- added R17: 100k, Resistor_SMD:R_0805_2012Metric_Pad1.15x1.40mm_HandSolder, B.Cu at (133.6, 112.0)
- added R18: 51k, Resistor_SMD:R_0805_2012Metric_Pad1.15x1.40mm_HandSolder, B.Cu at (133.6, 109.2)
- added R19: 18k, Resistor_SMD:R_0805_2012Metric_Pad1.15x1.40mm_HandSolder, B.Cu at (133.6, 114.8)
- added R2: 1k, Resistor_SMD:R_0805_2012Metric_Pad1.15x1.40mm_HandSolder, B.Cu at (134.1, 137.4)
- added R20: 100k, Resistor_SMD:R_0805_2012Metric_Pad1.15x1.40mm_HandSolder, B.Cu at (147.8, 116.1)
- added R21: 100k, Resistor_SMD:R_0805_2012Metric_Pad1.15x1.40mm_HandSolder, B.Cu at (147.8, 113.3)
- added R22: 68k, Resistor_SMD:R_0805_2012Metric_Pad1.15x1.40mm_HandSolder, B.Cu at (147.8, 110.5)
- added R23: 33k, Resistor_SMD:R_0805_2012Metric_Pad1.15x1.40mm_HandSolder, B.Cu at (147.8, 118.9)
- added R24: 2k2, Resistor_SMD:R_0805_2012Metric_Pad1.15x1.40mm_HandSolder, B.Cu at (152.1, 71.6)
- added R25: opt, Resistor_SMD:R_0805_2012Metric_Pad1.15x1.40mm_HandSolder, B.Cu at (144.5, 79.2)
- added R3: 1k, Resistor_SMD:R_0805_2012Metric_Pad1.15x1.40mm_HandSolder, B.Cu at (120.1, 137.4)
- added R4: 30k, Resistor_SMD:R_0805_2012Metric_Pad1.15x1.40mm_HandSolder, B.Cu at (115.3, 70.9)
- added R5: 150k, Resistor_SMD:R_0805_2012Metric_Pad1.15x1.40mm_HandSolder, B.Cu at (129.3, 70.9)
- added R6: 15k, Resistor_SMD:R_0805_2012Metric_Pad1.15x1.40mm_HandSolder, B.Cu at (118.1, 70.9)
- added R7: 30k, Resistor_SMD:R_0805_2012Metric_Pad1.15x1.40mm_HandSolder, B.Cu at (123.7, 70.9)
- added R8: 30k, Resistor_SMD:R_0805_2012Metric_Pad1.15x1.40mm_HandSolder, B.Cu at (120.9, 70.9)
- added R9: 30k, Resistor_SMD:R_0805_2012Metric_Pad1.15x1.40mm_HandSolder, B.Cu at (112.0, 70.9)
- added RV1: 100k, Potentiometer_THT:Potentiometer_Alpha_RD901F-40-00D_Single_Vertical, F.Cu at (129.5, 104.1)
- added RV2: 10k, Potentiometer_THT:Potentiometer_Alpha_RD901F-40-00D_Single_Vertical, F.Cu at (111.8, 66.0)
- added RV3: 5k, Potentiometer_THT:Potentiometer_Bourns_3296W_Vertical, B.Cu at (125.7, 121.2)
- added RV4: 10k, Potentiometer_THT:Potentiometer_Alpha_RD901F-40-00D_Single_Vertical, F.Cu at (147.3, 66.0)
- added RV5: 100k, Potentiometer_THT:Potentiometer_Alpha_RD901F-40-00D_Single_Vertical, F.Cu at (147.3, 104.1)
- added SW1: SW_DPDT_x2, svf_footprints:DPDT_on_on, F.Cu at (114.3, 96.5)
- added U1: TL072, Package_SO:SOIC-8_3.9x4.9mm_P1.27mm, B.Cu at (122.6, 78.2)
- added U2: SSM2164, Package_SO:SOIC-16_3.9x9.9mm_P1.27mm, B.Cu at (137.2, 78.2)
- added U3: TL072, Package_SO:SOIC-8_3.9x4.9mm_P1.27mm, B.Cu at (112.4, 78.2)
- added U4: TL072, Package_SO:SOIC-8_3.9x4.9mm_P1.27mm, B.Cu at (140.7, 119.6)
- added U5: LM4040DBZ-5, Package_TO_SOT_SMD:SOT-23_Handsoldering, B.Cu at (156.5, 70.1)
Routing:
- net -12V: track 0.00 -> 160.3 mm, vias 0 -> 4
- net +12V: track 0.00 -> 152.3 mm, vias 0 -> 3
- net /audio_path/band_pass_out: track 0.00 -> 124.0 mm, vias 0 -> 3
- net /audio_path/high_pass_out: track 0.00 -> 123.2 mm, vias 0 -> 2
- net /audio_path/low_pass_out: track 0.00 -> 89.2 mm, vias 0 -> 3
- net /audio_path/Vfc_in: track 0.00 -> 77.6 mm, vias 0 -> 3
- net Net-(C10-Pad2): track 0.00 -> 72.6 mm, vias 0 -> 1
- net Net-(C12-Pad2): track 0.00 -> 71.5 mm
- net /audio_path/filter_input: track 0.00 -> 67.2 mm, vias 0 -> 1
- net /audio_path/Vrez_in: track 0.00 -> 62.8 mm, vias 0 -> 2
- net Net-(C8-Pad2): track 0.00 -> 57.5 mm, vias 0 -> 3
- net -5V: track 0.00 -> 52.6 mm
- net Net-(C2-Pad1): track 0.00 -> 51.9 mm, vias 0 -> 4
- net Net-(C5-Pad2): track 0.00 -> 49.4 mm, vias 0 -> 3
- net Net-(C11-Pad2): track 0.00 -> 26.8 mm
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- added copper zone on B.Cu, net GND
- added copper zone on F.Cu, net GND
Other:
- board outline added: 58.4 x 99.1 mm
- rule pad_to_mask_clearance: 0.05 -> 0.051
- board text added: "1v/oct in"
- board text added: "1v/oct trim"
- board text added: "FM CV in"
- board text added: "band-pass out"
- board text added: "github.com/JordanAceto/SSM2164-SVF rev 0 2020-08-03"
- board text added: "gnd"
- board text added: "high-pass out"
- board text added: "low-pass out"
- board text added: "rez CV in"
- board text added: "signal in"
- board text added: "v+ in"
- board text added: "v- in"

Commit message: built and tested, minor component changes
Parts:
- C1: value 47pF -> dnf
- R5: value 150k -> 1M
Changed lines of the file:
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@@
-(kicad_pcb (version 20171130) (host pcbnew 5.1.6-c6e7f7d~87~ubuntu18.04.1)
+(kicad_pcb (version 20171130) (host pcbnew 5.1.7-a382d34a8~87~ubuntu18.04.1)
   (general
     (thickness 1.6)
@@
   )
   (setup
-    (last_trace_width 1)
+    (last_trace_width 0.25)
     (user_trace_width 0.29)
     (user_trace_width 0.4)
@@
     (visible_elements FFFFFF7F)
     (pcbplotparams
-      (layerselection 0x010fc_ffffffff)
+      (layerselection 0x010f0_ffffffff)
       (usegerberextensions false)
       (usegerberattributes false)
@@
       (psa4output false)
       (plotreference true)
-      (plotvalue true)
+      (plotvalue false)
       (plotinvisibletext false)
-      (padsonsilk false)
+      (padsonsilk true)
       (subtractmaskfromsilk false)
       (outputformat 1)
@@
       (effects (font (size 1 1) (thickness 0.15)))
     )
-    (fp_text user %R (at 0.3 0) (layer F.Fab)
-      (effects (font (size 1 1) (thickness 0.15)))
-    )
     (fp_circle (center 0 0) (end 3.2 0) (layer Cmts.User) (width 0.15))
     (fp_circle (center 0 0) (end 3.45 0) (layer F.CrtYd) (width 0.05))
+    (fp_text user %R (at 0.3 0) (layer F.Fab)
+      (effects (font (size 1 1) (thickness 0.15)))
+    )
     (pad 1 thru_hole circle (at 1.697056 -1.697056) (size 0.8 0.8) (drill 0.5) (layers *.Cu *.Mask)
       (net 2 GND))
@@
       (effects (font (size 1 1) (thickness 0.15)))
     )
-    (fp_text user %R (at 0.3 0) (layer F.Fab)
-      (effects (font (size 1 1) (thickness 0.15)))
-    )
     (fp_circle (center 0 0) (end 3.2 0) (layer Cmts.User) (width 0.15))
     (fp_circle (center 0 0) (end 3.45 0) (layer F.CrtYd) (width 0.05))
+    (fp_text user %R (at 0.3 0) (layer F.Fab)
+      (effects (font (size 1 1) (thickness 0.15)))
+    )
     (pad 1 thru_hole circle (at 1.697056 -1.697056) (size 0.8 0.8) (drill 0.5) (layers *.Cu *.Mask)
       (net 2 GND))
@@
       (effects (font (size 1 1) (thickness 0.15)) (justify mirror))
     )
-    (fp_text value 150k (at 0 -1.65 90) (layer B.Fab)
+    (fp_text value 1M (at 0 -1.65 90) (layer B.Fab)
       (effects (font (size 1 1) (thickness 0.15)) (justify mirror))
     )
@@
       (effects (font (size 1 1) (thickness 0.15)) (justify mirror))
     )
-    (fp_text value 47pF (at 0 -1.65 90) (layer B.Fab)
-      (effects (font (size 1 1) (thickness 0.15)) (justify mirror))
-    )
+    (fp_text value dnf (at 0 -1.65 90) (layer B.Fab)
+      (effects (font (size 1 1) (thickness 0.15)) (justify mirror))
+    )
