File: kicad_docs/audio_path.sch (KiCad schematic (older format))
At the start: 27 parts, among them SW1 SW_DPDT_x2, U1 TL072, U2 SSM2164, U3 TL072

Commit message: first rev pcb layout
Parts:
- C5, C6, C8, C9: footprint Capacitor_THT:C_Rect_L7.0mm_W4.5mm_P5.00mm -> svf_footprints:timing_cap_dual_fp
Connections:
- net GND: now also U2.10; no longer U2.15
- net Vrez_in: now also U2.14; no longer U2.11
- net low_pass_out: now also U3.7; no longer U3.1
- net at C2.1, R9.1: now also U2.13, U3.2 (-); no longer U2.12, U3.6 (-)
- net at C2.2, R6.1, R9.2: now also U3.1; no longer U3.7
- net at C8.2, C9.2, U2.5: now also U3.6 (-); no longer U3.2 (-)
- net at R12.2, R13.2: now also U2.15; no longer U2.10
Other:
- note added: "Integrator caps C5, C6, C8 and C9\nhave a dual footprint which can \naccept either through-hole or SMD\npackages. Fit only one or the other."
- note added: "Zeners D1 and D2 limit the\namplitude of the self oscillation.\n\nYou can experiment with different\nzeners or other clipping networks to\nachieve the desired sine wave amplitude\nwhen the filter is self oscillating.\n\nNote that these zeners also have some \ncapacitance which is in parallel with the\nintegrator cap(s). This may have some effect\non the filter. Experimentation is suggested."
- note added: "optional DPDT range switch\nadds 22nF in parallel with the\n220pF integrator caps which puts\nthe filter in very low frequency \nmode. When the switch is closed \nand the resonance is cranked\nup to the point of self-oscillation\nthe filter can be used as a sine \nwave LFO.\n\nIf this feature is not desired then\njust do not install C5, C8, and SW1."
- note removed: "optional DPDT range switch\nadds 22nF in parallel with the\n220pF integrator caps which puts\nthe filter in very low frequency \nmode. When the switch is closed \nand the resonance is cranked\nup to the point of self-oscillation\nthe filter can be used as a sine \nwave LFO."
- moved on the sheet: U2C, U2D, U3A, U3B
Changed lines of the file:
@@
 Connection ~ 2000 3450
-$Comp
-L Device:R R?
-U 1 1 5F726DEF
-P 3800 3700
-AR Path="/5F726DEF" Ref="R?"  Part="1"
-AR Path="/5F6F4121/5F726DEF" Ref="R11"  Part="1"
-F 0 "R11" H 3700 3700 50  0000 C CNN
-F 1 "510" V 3800 3700 50  0000 C CNN
-F 2 "Resistor_SMD:R_0805_2012Metric_Pad1.15x1.40mm_HandSolder" V 3730 3700 50  0001 C CNN
-F 3 "~" H 3800 3700 50  0001 C CNN
-	1    3800 3700
-	-1   0    0    1
-$EndComp
 $Comp
 L SSM2164_SVF_parts:SSM2164 U?
@@
 F 0 "C6" V 5498 3150 50  0000 C CNN
 F 1 "220pF" V 5589 3150 50  0000 C CNN
-F 2 "Capacitor_THT:C_Rect_L7.0mm_W4.5mm_P5.00mm" H 5788 3000 50  0001 C CNN
+F 2 "svf_footprints:timing_cap_dual_fp" H 5788 3000 50  0001 C CNN
 F 3 "~" H 5750 3150 50  0001 C CNN
 	1    5750 3150
@@
 F 0 "C5" V 5498 2350 50  0000 C CNN
 F 1 "22nF" V 5589 2350 50  0000 C CNN
-F 2 "Capacitor_THT:C_Rect_L7.0mm_W4.5mm_P5.00mm" H 5788 2200 50  0001 C CNN
+F 2 "svf_footprints:timing_cap_dual_fp" H 5788 2200 50  0001 C CNN
 F 3 "~" H 5750 2350 50  0001 C CNN
 	1    5750 2350
@@
 AR Path="/5F726E4B" Ref="R?"  Part="1"
 AR Path="/5F6F4121/5F726E4B" Ref="R15"  Part="1"
-F 0 "R15" H 7200 3700 50  0000 C CNN
+F 0 "R15" H 7150 3700 50  0000 C CNN
 F 1 "510" V 7300 3700 50  0000 C CNN
 F 2 "Resistor_SMD:R_0805_2012Metric_Pad1.15x1.40mm_HandSolder" V 7230 3700 50  0001 C CNN
@@
 L Amplifier_Operational:TL072 U?
 U 1 1 5F726E72
-P 9300 3550
+P 3000 6000
 AR Path="/5F726E72" Ref="U?"  Part="1"
 AR Path="/5F6F4121/5F726E72" Ref="U3"  Part="1"
-F 0 "U3" H 9400 3750 50  0000 C CNN
-F 1 "TL072" H 9450 3850 50  0000 C CNN
-F 2 "Package_SO:SOIC-8_3.9x4.9mm_P1.27mm" H 9300 3550 50  0001 C CNN
-F 3 "http://www.ti.com/lit/ds/symlink/tl071.pdf" H 9300 3550 50  0001 C CNN
-	1    9300 3550
-	1    0    0    1
+F 0 "U3" H 3100 6200 50  0000 C CNN
+F 1 "TL072" H 3150 6300 50  0000 C CNN
+F 2 "Package_SO:SOIC-8_3.9x4.9mm_P1.27mm" H 3000 6000 50  0001 C CNN
+F 3 "http://www.ti.com/lit/ds/symlink/tl071.pdf" H 3000 6000 50  0001 C CNN
+	1    3000 6000
+	-1   0    0    1
 $EndComp
 $Comp
@@
 F 0 "C9" V 9050 3150 50  0000 C CNN
 F 1 "220pF" V 9150 3150 50  0000 C CNN
-F 2 "Capacitor_THT:C_Rect_L7.0mm_W4.5mm_P5.00mm" H 9338 3000 50  0001 C CNN
+F 2 "svf_footprints:timing_cap_dual_fp" H 9338 3000 50  0001 C CNN
 F 3 "~" H 9300 3150 50  0001 C CNN
 	1    9300 3150
@@
 F 0 "C8" V 9050 2350 50  0000 C CNN
 F 1 "22nF" V 9150 2350 50  0000 C CNN
-F 2 "Capacitor_THT:C_Rect_L7.0mm_W4.5mm_P5.00mm" H 9338 2200 50  0001 C CNN
+F 2 "svf_footprints:timing_cap_dual_fp" H 9338 2200 50  0001 C CNN
 F 3 "~" H 9300 2350 50  0001 C CNN
 	1    9300 2350
@@
 L Amplifier_Operational:TL072 U?
 U 2 1 5F726EC1
-P 3000 6000
+P 9300 3550
 AR Path="/5F726EC1" Ref="U?"  Part="2"
 AR Path="/5F6F4121/5F726EC1" Ref="U3"  Part="2"
-F 0 "U3" H 3150 6150 50  0000 C CNN
-F 1 "TL072" H 3100 6250 50  0000 C CNN
-F 2 "Package_SO:SOIC-8_3.9x4.9mm_P1.27mm" H 3000 6000 50  0001 C CNN
-F 3 "http://www.ti.com/lit/ds/symlink/tl071.pdf" H 3000 6000 50  0001 C CNN
-	2    3000 6000
-	-1   0    0    1
+F 0 "U3" H 9450 3700 50  0000 C CNN
+F 1 "TL072" H 9400 3800 50  0000 C CNN
+F 2 "Package_SO:SOIC-8_3.9x4.9mm_P1.27mm" H 9300 3550 50  0001 C CNN
+F 3 "http://www.ti.com/lit/ds/symlink/tl071.pdf" H 9300 3550 50  0001 C CNN
+	2    9300 3550
+	1    0    0    1
 $EndComp
 $Comp
@@
 L SSM2164_SVF_parts:SSM2164 U?
 U 3 1 5F726EDD
-P 4700 5900
+P 10100 5850
 AR Path="/5F726EDD" Ref="U?"  Part="3"
 AR Path="/5F6F4121/5F726EDD" Ref="U2"  Part="3"
-F 0 "U2" H 4800 6265 50  0000 C CNN
-F 1 "SSM2164" H 4800 6174 50  0000 C CNN
-F 2 "Package_SO:SOIC-16_3.9x9.9mm_P1.27mm" H 4800 6100 50  0001 C CNN
-F 3 "" H 4800 6100 50  0001 C CNN
-	3    4700 5900
-	-1   0    0    -1
+F 0 "U2" H 10200 6215 50  0000 C CNN
+F 1 "SSM2164" H 10200 6124 50  0000 C CNN
+F 2 "Package_SO:SOIC-16_3.9x9.9mm_P1.27mm" H 10200 6050 50  0001 C CNN
+F 3 "" H 10200 6050 50  0001 C CNN
+	3    10100 5850
+	1    0    0    -1
 $EndComp
 Connection ~ 3400 5900
@@
 	4700 6400 4700 6200
 Text Notes 8850 1900 0    50   ~ 0
-optional DPDT range switch\nadds 22nF in parallel with the\n220pF integrator caps which puts\nthe filter in very low frequency \nmode. When the switch is closed \nand the resonance is cranked\nup to the point of self-oscillation\nthe filter can be used as a sine \nwave LFO.
+optional DPDT range switch\nadds 22nF in parallel with the\n220pF integrator caps which puts\nthe filter in very low frequency \nmode. When the switch is closed \nand the resonance is cranked\nup to the point of self-oscillation\nthe filter can be used as a sine \nwave LFO.\n\nIf this feature is not desired then\njust do not install C5, C8, and SW1.
 $Comp
 L SSM2164_SVF_parts:SSM2164 U?
 U 4 1 5F726F16
-P 10100 5850
+P 4700 5900
 AR Path="/5F726F16" Ref="U?"  Part="4"
 AR Path="/5F6F4121/5F726F16" Ref="U2"  Part="4"
-F 0 "U2" H 10100 6200 50  0000 C CNN
-F 1 "SSM2164" H 10100 6100 50  0000 C CNN
-F 2 "Package_SO:SOIC-16_3.9x9.9mm_P1.27mm" H 10200 6050 50  0001 C CNN
-F 3 "" H 10200 6050 50  0001 C CNN
-	4    10100 5850
-	1    0    0    -1
+F 0 "U2" H 4700 6250 50  0000 C CNN
+F 1 "SSM2164" H 4700 6150 50  0000 C CNN
+F 2 "Package_SO:SOIC-16_3.9x9.9mm_P1.27mm" H 4800 6100 50  0001 C CNN
+F 3 "" H 4800 6100 50  0001 C CNN
+	4    4700 5900
+	-1   0    0    -1
 $EndComp
 Text HLabel 2800 3100 2    50   Output ~ 0
@@
 NoConn ~ 10100 6150
 NoConn ~ 10600 5850
+Text Notes 6550 2650 0    50   ~ 0
+Integrator caps C5, C6, C8 and C9\nhave a dual footprint which can \naccept either through-hole or SMD\npackages. Fit only one or the other.
+Text Notes 5200 1900 0    50   ~ 0
+Zeners D1 and D2 limit the\namplitude of the self oscillation.\n\nYou can experiment with different\nzeners or other clipping networks to\nachieve the desired  sine wave amplitude\nwhen the filter is self oscillating.\n\nNote that these zeners also have some \ncapacitance which is in parallel with the\nintegrator cap(s). This may have some effect\non the filter. Experimentation is suggested.
+$Comp
+L Device:R R?
+U 1 1 5F726DEF
+P 3800 3700
+AR Path="/5F726DEF" Ref="R?"  Part="1"
+AR Path="/5F6F4121/5F726DEF" Ref="R11"  Part="1"
+F 0 "R11" H 3650 3700 50  0000 C CNN
+F 1 "510" V 3800 3700 50  0000 C CNN
+F 2 "Resistor_SMD:R_0805_2012Metric_Pad1.15x1.40mm_HandSolder" V 3730 3700 50  0001 C CNN
+F 3 "~" H 3800 3700 50  0001 C CNN
+	1    3800 3700
+	-1   0    0    1
+$EndComp
 $EndSCHEMATC

Commit message: built and tested, minor component changes
Parts:
- C1: value 47pF -> dnf
- R5: value 150k -> 1M
Changed lines of the file:
@@
 AR Path="/5F6F4121/5F726EAB" Ref="R5"  Part="1"
 F 0 "R5" V 2250 4600 50  0000 C CNN
-F 1 "150k" V 2350 4600 50  0000 C CNN
+F 1 "1M" V 2350 4600 50  0000 C CNN
 F 2 "Resistor_SMD:R_0805_2012Metric_Pad1.15x1.40mm_HandSolder" V 2280 4600 50  0001 C CNN
 F 3 "~" H 2350 4600 50  0001 C CNN
@@
 AR Path="/5F6F4121/5F2E065B" Ref="C1"  Part="1"
 F 0 "C1" V 2148 1600 50  0000 C CNN
-F 1 "47pF" V 2239 1600 50  0000 C CNN
+F 1 "dnf" V 2239 1600 50  0000 C CNN
 F 2 "Capacitor_SMD:C_0805_2012Metric_Pad1.15x1.40mm_HandSolder" H 2438 1450 50  0001 C CNN
 F 3 "~" H 2400 1600 50  0001 C CNN
